Commit message: changed gripper to not use mimic removed gazebo stuff

File: egh_gripper_description/urdf/egh_gripper.urdf.xacro (robot description, xacro)
@@ -45,14 +45,4 @@
             <dynamics friction="100" damping="100" />
         </joint>
-        <transmission name="${prefix}_base_trans_left">
-            <type>transmission_interface/SimpleTransmission</type>
-            <actuator name="${prefix}_base_motor_left">
-                <mechanicalReduction>1</mechanicalReduction>
-                <motorTorqueConstant>1</motorTorqueConstant>
-            </actuator>
-            <joint name="${prefix}_finger_left_joint" >
-                <hardwareInterface>hardware_interface/PositionJointInterface</hardwareInterface>
-            </joint>
-        </transmission>
         <link name="${prefix}_left_finger">
             <inertial>
@@ -68,6 +58,6 @@
                     <mesh filename="package://egh_gripper_description/meshes/egh_finger.stl" scale="1.0 1.0 1.0"/>
                 </geometry>
-                <material name="black">
-                <color rgba="0 0 0 0"/>
+                <material name="grey">
+                <color rgba="0.5 0.5 0.5 1"/>
                 </material>
             </visual>
@@ -80,8 +70,4 @@
             <contact_coefficients kd="1.0" kp="1000.0" mu="0"/>
         </link>
-        <gazebo reference="${prefix}_left_finger">
-            <material>Gazebo/Blue</material>
-            <turnGravityOff>false</turnGravityOff>
-        </gazebo>
         <!-- FINGER RIGHT -->
         <joint name="${prefix}_finger_right_joint" type="prismatic">
@@ -92,41 +78,5 @@
             <child link="${prefix}_right_finger" />
             <dynamics friction="100" damping="100" />
-            <mimic joint="${prefix}_finger_left_joint" multiplier="1" offset="0"/>
         </joint>
-        <!--
-            The transmission is not defined cause the right finger is mirroring
-            the left finger using mimic plugin
-        -->
-        <!--transmission name="${prefix}_base_trans_right">
-            <type>transmission_interface/SimpleTransmission</type>
-            <actuator name="${prefix}_base_motor_right">
-                <mechanicalReduction>1</mechanicalReduction>
-                <motorTorqueConstant>1</motorTorqueConstant>
-            </actuator>
-            <joint name="${prefix}_finger_right_joint" >
-                <hardwareInterface>hardware_interface/PositionJointInterface</hardwareInterface>
-            </joint>
-        </transmission-->
-        <xacro:macro name="mimic_joint_plugin_gazebo" params="parent_joint mimic_joint has_pid:=false multiplier:=1.0 offset:=0 sensitiveness:=0.0 max_effort:=1.0 robot_namespace:=''">
-            <gazebo>
-                <plugin name="${mimic_joint}_mimic_joint_plugin" filename="libroboticsgroup_gazebo_mimic_joint_plugin.so">
-                    <joint>${parent_joint}</joint>
-                    <mimicJoint>${mimic_joint}</mimicJoint>
-                    <xacro:if value="${has_pid}">
-                    <hasPID />
-                    </xacro:if>
-                    <multiplier>${multiplier}</multiplier>
-                    <offset>${offset}</offset>
-                    <sensitiveness>${sensitiveness}</sensitiveness>
-                    <maxEffort>${max_effort}</maxEffort>
-                    <xacro:unless value="${robot_namespace == ''}">
-                        <robotNamespace>($robot_namespace)</robotNamespace>
-                    </xacro:unless>
-                </plugin>
-            </gazebo>
-        </xacro:macro>
-        <xacro:mimic_joint_plugin_gazebo parent_joint="${prefix}_finger_left_joint"
-        mimic_joint="${prefix}_finger_right_joint" has_pid="false" multiplier="1.0"
-        max_effort="10.0" />
         <link name="${prefix}_right_finger">
             <inertial>
@@ -142,6 +92,6 @@
                     <mesh filename="package://egh_gripper_description/meshes/egh_finger.stl" scale="1.0 1.0 1.0"/>
                 </geometry>
-                <material name="black">
-                <color rgba="0 0 0 0"/>
+                <material name="grey">
+                <color rgba="0.5 0.5 0.5 1"/>
                 </material>
             </visual>
